File: analog-sidequest/stage0_5-hardware/Stage0_5.kicad_sch (KiCad schematic)
At the start: 71 parts, among them J1 302-S401, U1 MCP4251-103E-SL, U10 AMS1117-3.3, U11 OPA2333AIDGKTG4, U12 OPA2333AIDGKTG4, U13 OPA2333AIDGKTG4, U2 MCP4251-103E-SL, U3 MCP4251-103E-SL, U4 MCP4251-103E-SL, U5 MCP4251-103E-SL, U6 MCP4251-103E-SL, U7 SN74HC138PWR, U8 MCP4728A0T-E/UN, U9 ADS1115IDGSR

Commit message: Stage 0.5 hardware: rename to Stage0_5, drop orphans, add silkscreen logo
The KiCad project renamed Effective_Black_R2-D2 → Stage0_5 (the
canonical name; the original was KiCad's auto-generated random name).
KiCad's File → Save As propagated the rename to the schematic, PCB,
project, custom symbols, netlist, design-notes sidecar, BOM CSV, and
the gerber zip in gerber_to_order/. Git records these as renames.

Two architectural fixes the user landed during the rename pass and
that this commit captures via the renamed files:

 * R7 and R10 in the schematic are now spec'd as `10k 0.1%` instead
   of the generic 1% Yageo. Those are the two combiner-input
   positions paired with R24/R25 (2.56 MΩ 0.1%) for the binary-
   weighted 1:1/256 ratio. Without that swap, the ratio precision
   was limited to ~1% — about 18× the σ ≈ 6e-4 RMS noise budget.
 * Every R and C `Value` field is now populated with a real value
   ("10k", "10k 0.1%", "40k 0.1%", "2.56M 0.1%", "4.7k", "13Ω 5%",
   "100nF", "10uF") instead of "Generic Resistor" / "Generic
   Capacitor". Silkscreen, BOM, and ERC stay in sync now.

Cleanup:
 * Untitled.kicad_mod orphan removed (the new Stage0_5 PCB does not
   reference it; verified by grep).
 * stage0_5-harware-docs/ (the typo'd sidecar with the original
   project notes) removed; its content is superseded by
   Stage0_5-design-notes.md and the canonical STAGE0_5.md spec doc
   one level up.
 * Two stale Effective_Black_R2-D2-*.csv / .md files that KiCad's
   Save As did not auto-delete — manually removed from the working
   tree.
 * Old Effective_Black_R2-D2-all-pos.csv and stage0.cpl.numbers /
   stage0.csv assembly files in gerber_to_order/ removed alongside
   the corresponding renamed gerber zip.

New asset:
 * analog-sidequest/silkscreen/logo35x14.kicad_mod — silkscreen logo
   footprint for the board. The PNG source images used to generate
   it (ChatGPT-rendered) are intentionally not tracked; the .mod is
   the deliverable.

Co-Authored-By: Claude O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
Parts:
- C1, C11, C12, C13, C14, C2, C3, C4, C5, C6, C7, C8, C9: value Capacitor 100 nF -> 100nF
- C10: value Capacitor 10 µF -> 100nF
- C15, C16, C17, C18, C19, C20: value Capacitor 100 nF -> 10uF
- R1, R11, R2, R3, R4, R5, R6, R8, R9: value Generic Resistor -> 10k
- R10, R7: value Generic Resistor -> 10k 0.1%
- R12, R13, R14, R15, R16, R17, R18, R19, R20, R21, R22, R23: value Generic Resistor -> 40k 0.1%
- R24, R25: value Generic Resistor -> 2.56M 0.1%
- R26, R27: value Matched Pair Resistor 10 kΩ -> 4.7k
- R28: value Generic Resistor -> 13Ω 5%
- U1, U2, U3, U4, U5, U6: value MCP4251-103E-SL -> MCP4251-103E/SL
Other:
- title: Effective_Black_R2-D2 -> Stage0_5
